File: tattoo_machine_power_bank.kicad_sch (KiCad schematic)
At the start: 230 parts, among them J1 Jack-DC, J2 IN_BAT_POWERBANK, J3 USB_C_Receptacle, J4 USB_A, J5 IN_BATCONTROL, J6 PROGRAM_SW, Q1 AOD403, Q10 A03420, Q11 MTB3904, Q12 A03420, Q13 2N7002, Q2 AOD403, Q3 AOD403, Q4 IRFN3709, Q5 IRFN3709, Q6 A03420, Q7 A03420, Q8 NPN, Q9 NPN, SW1 SW_Push, SW2 SW_Push, U1 STM32L010C6Tx, U10 TP181, U11 TP181, U12 TP181, U14 RT9193, U2 BQ24610, U3 RT9193, U4 IP5306, U5 SW6208, U6 SSD1327, U7 SX1308, U8 XB8688, U9 XB8688, Y1 8MHz

Commit message: sua file
Parts:
- removed JP5, JP6, JP7, JP8: OPEN FOR I2C, symbol Jumper:SolderJumper_2_Open
Changed lines of the file:
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@@
     (stroke (width 0) (type default))
   )
-  (wire (pts (xy 396.875 332.74) (xy 411.48 332.74))
-    (stroke (width 0) (type default))
-  )
   (wire (pts (xy 63.5 199.39) (xy 63.5 196.85))
     (stroke (width 0) (type default))
@@
     (stroke (width 0) (type default))
   )
-  (wire (pts (xy 374.65 332.74) (xy 389.255 332.74))
-    (stroke (width 0) (type default))
-  )
   (wire (pts (xy 132.08 284.48) (xy 132.08 285.75))
     (stroke (width 0) (type default))
@@
     (stroke (width 0) (type default))
   )
-  (wire (pts (xy 375.92 353.695) (xy 390.525 353.695))
-    (stroke (width 0) (type default))
-  )
   (wire (pts (xy 271.145 394.335) (xy 274.32 394.335))
     (stroke (width 0) (type default))
@@
     (stroke (width 0) (type default))
   )
-  (wire (pts (xy 398.145 351.155) (xy 412.75 351.155))
-    (stroke (width 0) (type default))
-  )
   (wire (pts (xy 118.11 342.265) (xy 117.475 342.265))
     (stroke (width 0) (type default))
@@
     (stroke (width 0) (type default))
   )
-  (wire (pts (xy 374.65 335.28) (xy 389.255 335.28))
-    (stroke (width 0) (type default))
-  )
   (wire (pts (xy 262.89 81.28) (xy 265.43 81.28))
     (stroke (width 0) (type default))
@@
     (stroke (width 0) (type default))
   )
-  (wire (pts (xy 396.875 335.28) (xy 411.48 335.28))
-    (stroke (width 0) (type default))
-  )
   (wire (pts (xy 379.73 205.74) (xy 379.73 208.28))
     (stroke (width 0) (type default))
@@
     (stroke (width 0) (type default))
   )
-  (wire (pts (xy 398.145 353.695) (xy 412.75 353.695))
-    (stroke (width 0) (type default))
-  )
   (wire (pts (xy 325.12 83.82) (xy 325.12 87.63))
     (stroke (width 0) (type default))
@@
     (stroke (width 0) (type default))
   )
-  (wire (pts (xy 375.92 351.155) (xy 390.525 351.155))
-    (stroke (width 0) (type default))
-  )
   (wire (pts (xy 129.54 60.96) (xy 129.54 63.5))
     (stroke (width 0) (type default))
@@
     (effects (font (size 1 1)) (justify left bottom))
   )
-  (label "D0_SPI_SCK{slash}I2C_SCL" (at 398.145 332.74 0) (fields_autoplaced)
-    (effects (font (size 1 1)) (justify left bottom))
-  )
   (label "ADC7_AVABTCONTROL" (at 245.745 394.335 0) (fields_autoplaced)
     (effects (font (size 1 1)) (justify left bottom))
@@
     (effects (font (size 1 1)) (justify left bottom))
   )
-  (label "D1_SPI_SDI{slash}I2C_SDA" (at 398.145 335.28 0) (fields_autoplaced)
-    (effects (font (size 1 1)) (justify left bottom))
-  )
   (label "NTC" (at 86.36 186.69 0) (fields_autoplaced)
     (effects (font (size 1 1)) (justify left bottom))
@@
     (effects (font (size 1 1)) (justify left bottom))
   )
-  (label "I2C1_SDA" (at 376.555 335.28 0) (fields_autoplaced)
-    (effects (font (size 1 1)) (justify left bottom))
-  )
-  (label "I2C1_SCL" (at 376.555 332.74 0) (fields_autoplaced)
-    (effects (font (size 1 1)) (justify left bottom))
-  )
   (label "KEY_IP5306" (at 69.85 349.25 90) (fields_autoplaced)
     (effects (font (size 1 1)) (justify left bottom))
   )
-  (label "D1_SPI_SDI{slash}I2C_SDA" (at 399.415 353.695 0) (fields_autoplaced)
-    (effects (font (size 1 1)) (justify left bottom))
-  )
   (label "SPI1_MOSI" (at 346.71 198.12 0) (fields_autoplaced)
     (effects (font (size 1 1)) (justify left bottom))
@@
     (effects (font (size 1 1)) (justify left bottom))
   )
-  (label "SPI1_SCK" (at 377.825 351.155 0) (fields_autoplaced)
-    (effects (font (size 1 1)) (justify left bottom))
-  )
   (label "SW_DIO" (at 491.49 226.06 0) (fields_autoplaced)
     (effects (font (size 1 1)) (justify left bottom))
@@
     (effects (font (size 1 1)) (justify left bottom))
   )
-  (label "SPI1_MOSI" (at 377.825 353.695 0) (fields_autoplaced)
-    (effects (font (size 1 1)) (justify left bottom))
-  )
   (label "DMA1" (at 144.78 274.32 0) (fields_autoplaced)
     (effects (font (size 1 1)) (justify left bottom))
@@
     (effects (font (size 1 1)) (justify left bottom))
   )
-  (label "D0_SPI_SCK{slash}I2C_SCL" (at 399.415 351.155 0) (fields_autoplaced)
-    (effects (font (size 1 1)) (justify left bottom))
-  )
   (label "ADC5_AVUSBA1" (at 396.875 142.24 0) (fields_autoplaced)
     (effects (font (size 1 1)) (justify left bottom))
@@
     )
   )
-  (symbol (lib_id "Jumper:SolderJumper_2_Open") (at 393.065 332.74 180) (unit 1)
-    (in_bom yes) (on_board yes) (dnp no)
-    (property "Reference" "JP5" (at 389.255 329.565 0)
-      (effects (font (size 1 1)))
-    )
-    (property "Value" "OPEN FOR I2C" (at 396.875 329.565 0)
-      (effects (font (size 1 1)))
-    )
-    (property "Footprint" "" (at 393.065 332.74 0)
-      (effects (font (size 1 1)) hide)
-    )
-    (property "Datasheet" "~" (at 393.065 332.74 0)
-      (effects (font (size 1 1)) hide)
-    )
-    (pin "1")
-    (pin "2")
-    (instances
-      (project "tattoo_machine_power_bank"
-        (path "/33716a33-1e59-4dba-bca6-adcfcc42978d"
-          (reference "JP5") (unit 1)
-        )
-      )
-    )
-  )
   (symbol (lib_id "Device:R_Small") (at 528.955 282.575 90) (unit 1)
     (in_bom yes) (on_board yes) (dnp no)
@@
     )
   )
-  (symbol (lib_id "Jumper:SolderJumper_2_Open") (at 394.335 353.695 180) (unit 1)
-    (in_bom yes) (on_board yes) (dnp no)
-    (property "Reference" "JP8" (at 389.89 357.505 0)
-      (effects (font (size 1 1)))
-    )
-    (property "Value" "OPEN FOR I2C" (at 397.51 357.505 0)
-      (effects (font (size 1 1)))
-    )
-    (property "Footprint" "" (at 394.335 353.695 0)
-      (effects (font (size 1 1)) hide)
-    )
-    (property "Datasheet" "~" (at 394.335 353.695 0)
-      (effects (font (size 1 1)) hide)
-    )
-    (pin "1")
-    (pin "2")
-    (instances
-      (project "tattoo_machine_power_bank"
-        (path "/33716a33-1e59-4dba-bca6-adcfcc42978d"
-          (reference "JP8") (unit 1)
-        )
-      )
-    )
-  )
   (symbol (lib_id "Device:R_Small") (at 41.275 337.185 180) (unit 1)
     (in_bom yes) (on_board yes) (dnp no)
@@
     )
   )
-  (symbol (lib_id "Jumper:SolderJumper_2_Open") (at 393.065 335.28 180) (unit 1)
-    (in_bom yes) (on_board yes) (dnp no)
-    (property "Reference" "JP6" (at 389.255 339.09 0)
-      (effects (font (size 1 1)))
-    )
-    (property "Value" "OPEN FOR I2C" (at 396.875 339.09 0)
-      (effects (font (size 1 1)))
-    )
-    (property "Footprint" "" (at 393.065 335.28 0)
-      (effects (font (size 1 1)) hide)
-    )
-    (property "Datasheet" "~" (at 393.065 335.28 0)
-      (effects (font (size 1 1)) hide)
-    )
-    (pin "1")
-    (pin "2")
-    (instances
-      (project "tattoo_machine_power_bank"
-        (path "/33716a33-1e59-4dba-bca6-adcfcc42978d"
-          (reference "JP6") (unit 1)
-        )
-      )
-    )
-  )
   (symbol (lib_id "Simulation_SPICE:NMOS") (at 236.22 82.55 0) (unit 1)
     (in_bom yes) (on_board yes) (dnp no) (fields_autoplaced)
@@
         )
       )
-    )
-  )
-  (symbol (lib_id "Jumper:SolderJumper_2_Open") (at 394.335 351.155 180) (unit 1)
-    (in_bom yes) (on_board yes) (dnp no)
-    (property "Reference" "JP7" (at 390.525 348.615 0)
-      (effects (font (size 1 1)))
-    )
-    (property "Value" "OPEN FOR I2C" (at 398.145 348.615 0)
-      (effects (font (size 1 1)))
-    )
-    (property "Footprint" "" (at 394.335 351.155 0)
-      (effects (font (size 1 1)) hide)
-    )
-    (property "Datasheet" "~" (at 394.335 351.155 0)
-      (effects (font (size 1 1)) hide)
-    )
-    (pin "1")
-    (pin "2")
-    (instances
-      (project "tattoo_machine_power_bank"
-        (path "/33716a33-1e59-4dba-bca6-adcfcc42978d"
-          (reference "JP7") (unit 1)
-        )
-      )
